File: fsckpad-hardware/fsckpad-hardware.kicad_sch (KiCad schematic)
At the start: 36 parts, among them J1 UART Socket, SW1 SW_Push_45deg, SW10 SW_Push_45deg, SW11 SW_Push_45deg, SW12 SW_Push_45deg, SW13 SW_Push, SW14 SW_Push, SW15 SW_Push_45deg, SW16 SW_Push_45deg, SW17 SW_Push_45deg, SW2 SW_Push_45deg, SW3 SW_Push_45deg, SW4 SW_Push_45deg, SW5 SW_Push_45deg, SW6 SW_Push_45deg, SW7 SW_Push_45deg, SW8 SW_Push_45deg, SW9 SW_Push_45deg, U1 COM-09032, U1 PCA9555D, U2 CR2013-MI2120, U3 A1301EUA-T, U4 A1301EUA-T, U5 MPU-9150, U6 COM-09032

Commit message: Revision 1.0 with haptic driver
Parts:
- removed H10: Touch R, symbol Mechanical:MountingHole_Pad_MP
- removed H6, H7, H8: MountingHole, MountingHole:MountingHole_3.2mm_M3_DIN965, symbol Mechanical:MountingHole
- removed H9: Touch L, symbol Mechanical:MountingHole_Pad_MP
- removed J1: UART Socket, symbol Connector:Conn_01x06_Socket
- removed SW10, SW11, SW12, SW15, SW16, SW17, SW5, SW6, SW7, SW8, SW9: SW_Push_45deg, symbol Switch:SW_Push_45deg
- removed SW13, SW14: SW_Push, symbol Switch:SW_Push
- removed U2: CR2013-MI2120, Display:CR2013-MI2120, symbol Driver_Display:CR2013-MI2120
- removed U5: MPU-9150, Sensor_Motion:InvenSense_QFN-24_4x4mm_P0.5mm, symbol Sensor_Motion:MPU-9150
- added A1, B1, POW1, X1, Y1: 1-TS009, JSP_Footprints:SW_Push_1TS009_Conductive_Pad, symbol Switch:SW_Push_45deg
- added Bite1, Bite2: Fiducial, JSP_Footprints:6.5mm_MouseBite, symbol Mechanical:Fiducial
- added C1: 0.1 uf, Capacitor_SMD:C_0603_1608Metric_Pad1.08x0.95mm_HandSolder, symbol Device:C
- added C2: 2.2 uf, Capacitor_SMD:C_0603_1608Metric_Pad1.08x0.95mm_HandSolder, symbol Device:C
- added C3: 10 nf, Capacitor_SMD:C_0603_1608Metric_Pad1.08x0.95mm_HandSolder, symbol Device:C
- added C4: 1 pF, Capacitor_SMD:C_0603_1608Metric_Pad1.08x0.95mm_HandSolder, symbol Device:C
- added C5: 1 pF, Capacitor_SMD:C_0603_1608Metric_Pad1.08x0.95mm_HandSolder, symbol Device:C_Small
- added Centroid1: Fiducial, Symbol:OSHW-Logo2_7.3x6mm_SilkScreen, symbol Mechanical:Fiducial
- added EYESPI1: Conn_01x18_Pin, Connector_FFC-FPC:Hirose_FH12-18S-0.5SH_1x18-1MP_P0.50mm_Horizontal, symbol Connector:Conn_01x18_Pin
- added Ext1: H1, Connector_PinHeader_1.00mm:PinHeader_2x02_P1.00mm_Vertical, symbol Connector_Generic:Conn_02x02_Odd_Even
- added Ext4: Conn_02x07_Counter_Clockwise, Connector_PinHeader_1.00mm:PinHeader_2x06_P1.00mm_Vertical, symbol Connector_Generic:Conn_02x06_Odd_Even
- added Ext5: Conn_02x02_Top_Bottom, Connector_PinHeader_1.00mm:PinHeader_2x02_P1.00mm_Vertical, symbol Connector_Generic:Conn_02x02_Odd_Even
- added IC1, IC6: LS20-S, digikey-kicad-library:SOIC-20_W7.5mm, symbol LS20-S:LS20-S
- added IC3: ICM-42670-P, ICM-42670-P:XDCR_ICM-42670-P, symbol ICM-42670-P:ICM-42670-P
- added IC5: PCA9555D, Package_SO:SOIC-24W_7.5x15.4mm_P1.27mm, symbol Interface_Expansion:PCA9555D
- added LB1, RB1: PTS645V, Button_Switch_THT:SW_Tactile_SPST_Angled_PTS645Vx39-2LFS, symbol Switch:SW_Push_45deg
- added LPDL1, RPDL1: 1-TS009, Button_Switch_SMD:SW_Push_1P1T_NO_6x6mm_H9.5mm, symbol Switch:SW_Push_45deg
- added LRA/ERM1: Conn_02x02_Odd_Even, Connector_PinHeader_1.00mm:PinHeader_2x02_P1.00mm_Vertical, symbol Connector_Generic:Conn_02x02_Odd_Even
- added LRAEnable1: 0, Jumper:SolderJumper-2_P1.3mm_Open_TrianglePad1.0x1.5mm, symbol Device:R
- added LTouch1, RTouch1: Conn_01x01_Pin, Connector_PinHeader_1.00mm:PinHeader_1x01_P1.00mm_Vertical, symbol Connector:Conn_01x01_Pin
- added Mate1: Conn_01x13, JSP_Footprints:BridgeableComb_1x13_Reverse, symbol Connector_Generic:Conn_01x13
- added PSOrient1, XBOrient1: Conn_01x13, JSP_Footprints:BridgeableComb_1x13, symbol Connector_Generic:Conn_01x13
- added R1, R2: 1M, Resistor_SMD:R_0603_1608Metric_Pad0.98x0.95mm_HandSolder, symbol Device:R_45deg
- added R4, R5: 10k, Resistor_SMD:R_0603_1608Metric_Pad0.98x0.95mm_HandSolder, symbol Device:R
- added STEMMA-QT1: Conn_01x04, Connector_JST:JST_SH_SM04B-SRSS-TB_1x04-1MP_P1.00mm_Horizontal, symbol Connector_Generic:Conn_01x04
- added Select1, Start1: 1-TS009, JSP_Footprints:SW_Push_1TS009_Conductive_Pad, symbol Switch:SW_Push
- added U1: DRV2605LDGS, Package_SO:VSSOP-10_3x3mm_P0.5mm, symbol Driver_Haptic:DRV2605LDGS
- +D1: renamed from SW4; value SW_Push_45deg -> 1-TS009; footprint (none) -> JSP_Footprints:SW_Push_1TS009_Conductive_Pad
- +L1: renamed from SW2; value SW_Push_45deg -> 1-TS009; footprint (none) -> JSP_Footprints:SW_Push_1TS009_Conductive_Pad
- +R1: renamed from SW3; value SW_Push_45deg -> 1-TS009; footprint (none) -> JSP_Footprints:SW_Push_1TS009_Conductive_Pad
- +U1: renamed from SW1; value SW_Push_45deg -> 1-TS009; footprint (none) -> JSP_Footprints:SW_Push_1TS009_Conductive_Pad
- H1, H2, H3, H4, H5: footprint MountingHole:MountingHole_3.2mm_M3_DIN965 -> MountingHole:MountingHole_2.7mm_M2.5_DIN965; now left out of the parts list
- LS1: renamed from U1; footprint XDCR_COM-09032 -> COM-09032:XDCR_COM-09032
- LT1: renamed from U3; footprint (none) -> Package_TO_SOT_THT:TO-92Flat
- RS1: renamed from U6; footprint XDCR_COM-09032 -> COM-09032:XDCR_COM-09032
- RT1: renamed from U4; footprint (none) -> Package_TO_SOT_THT:TO-92Flat
- renumbered U1 to IC4, A1 to M1
Connections:
- net +3.3V: now also M1.2 (3V3), C1.2, C2.2, C3.2, C4.1, EYESPI1.1 (Pin_1), IC1.1 (VDD), IC3.12 (AP_CS), IC3.5 (VDDIO), IC3.8 (VDD), IC5.21 (A0), IC5.24 (VDD), IC6.1 (VDD), Mate1.8 (Pin_8), PSOrient1.8 (Pin_8), R4.2, R5.2, STEMMA-QT1.2 (Pin_2), U1.10 (VDD), U1.5 (EN), U1.6 (VDD/NC), XBOrient1.8 (Pin_8)
- net GND: now also +D1.1, +L1.1, +R1.1, +U1.1, A1.1, B1.1, C1.1, C2.1, C3.1, C4.2, C5.2, EYESPI1.3 (Pin_3), Ext1.2 (Pin_2), Ext1.4 (Pin_4), Ext4.1 (Pin_1), Ext4.11 (Pin_11), Ext4.3 (Pin_3), Ext4.5 (Pin_5), Ext4.7 (Pin_7), Ext4.9 (Pin_9), Ext5.2 (Pin_2), Ext5.4 (Pin_4), IC1.20 (VSS), IC3.1 (AP_SDO/AP_AD0), IC3.10 (RESV), IC3.11 (RESV), IC3.2 (RESV), IC3.3 (RESV), IC3.6 (GND), IC3.7 (FSYNC), IC5.12 (VSS), IC5.2 (A1), IC5.3 (A2), IC6.20 (VSS), LB1.1, LPDL1.1, LRAEnable1.2, Mate1.7 (Pin_7), POW1.1, PSOrient1.7 (Pin_7), RB1.1, RPDL1.1, STEMMA-QT1.1 (Pin_1), Select1.2, Start1.2, U1.4 (IN/TRIG), U1.8 (GND), X1.1, XBOrient1.6 (Pin_6), XBOrient1.7 (Pin_7), Y1.1
- net at IC4.7 (IO0_3): now also IC1.16 (OUT3); no longer +D1.2
- net LT: now reaches LT1.3 (VOUT)
- net LT: now also M1.7 (A2); no longer M1.10 (A5)
- net LTouchProbe: now reaches IC4.19 (IO1_6)
- net LTouchProbe: now also Mate1.13 (Pin_13), PSOrient1.13 (Pin_13), R2.1, XBOrient1.13 (Pin_13); no longer RS1.B1A (SEL+)
- net LJSH: now reaches M1.5 (A0)
- net LJSH: now also LS1.H2 (H), Mate1.10 (Pin_10), PSOrient1.10 (Pin_10), XBOrient1.10 (Pin_10); no longer RS1.H2 (H)
- net LJSV: now reaches M1.6 (A1)
- net LJSV: now also LS1.V2 (V), Mate1.11 (Pin_11), PSOrient1.11 (Pin_11), XBOrient1.11 (Pin_11); no longer RS1.V2 (V)
- net at IC4.5 (IO0_1): now also IC1.18 (OUT1); no longer +L1.2
- net at IC4.4 (IO0_0): now also IC1.19 (OUT0); no longer +U1.2
- net at IC4.10 (IO0_6): now also IC1.13 (OUT6)
- net at IC4.6 (IO0_2): now also IC1.17 (OUT2); no longer +R1.2
- net LJSS: now reaches LS1.B1A (SEL+)
- net LJSS: now also IC1.8 (SW6), Mate1.9 (Pin_9), PSOrient1.9 (Pin_9), XBOrient1.9 (Pin_9); no longer IC4.20 (IO1_7)
- net RT: now reaches M1.8 (A3)
- net RT: now also RT1.3 (VOUT); no longer LS1.V2 (V)
- net at IC4.13 (IO1_0): now also IC1.11 (OUT8)
- net at IC4.8 (IO0_4): now also IC1.15 (OUT4)
- net at M1.12 (MOSI): now also EYESPI1.5 (Pin_5)
- net at M1.11 (SCK): now also EYESPI1.4 (Pin_4)
- net at M1.13 (MISO): now also EYESPI1.6 (Pin_6)
- net at M1.19 (D5): now also EYESPI1.9 (Pin_9); no longer IC4.1 (~{INT})
- net at IC4.11 (IO0_7): now also IC1.12 (OUT7)
- net at IC4.14 (IO1_1): now also Select1.1
- net LRASelect: now reaches IC4.15 (IO1_2)
- net LRASelect: now also LRAEnable1.1
- net SCL: now reaches IC4.22 (SCL), M1.18 (SCL)
- net SCL: now also EYESPI1.13 (Pin_13), IC3.13 (AP_SCL/AP_SCLK), IC5.22 (SCL), R4.1, STEMMA-QT1.4 (Pin_4), U1.2 (SCL)
- net SDA: now reaches IC4.23 (SDA), M1.17 (SDA)
- net SDA: now also EYESPI1.14 (Pin_14), IC3.14 (AP_SDA/AP_SDIO/AP_SDI), IC5.23 (SDA), R5.1, STEMMA-QT1.3 (Pin_3), U1.3 (SDA)
- net at IC4.9 (IO0_5): now also IC1.14 (OUT5)
- net RESET: now reaches M1.1 (~{RESET})
- net RESET: now also EYESPI1.8 (Pin_8)
- net at M1.14 (RX): now also EYESPI1.12 (Pin_12)
- net at M1.15 (TX): now also EYESPI1.2 (Pin_2)
- net RTouchSense: now reaches M1.16 (D2)
- net RTouchSense: now also R1.2, RTouch1.1 (Pin_1)
- net at M1.20 (D6): now also EYESPI1.7 (Pin_7)
- net PS: now reaches M1.21 (D7)
- net PS: now also POW1.2
- net D8: now reaches M1.22 (D8)
- net D8: now also Ext1.1 (Pin_1)
- net D9: now reaches M1.23 (D9)
- net D9: now also Ext1.3 (Pin_3)
- net INTERRUPT: now reaches M1.24 (D10)
- net INTERRUPT: now also IC4.1 (~{INT}), EYESPI1.15 (Pin_15), IC3.4 (INT1/INT), IC3.9 (INT2), IC5.1 (~{INT})
- net LTouchSense: now reaches M1.25 (D11)
- net LTouchSense: now also LTouch1.1 (Pin_1), Mate1.12 (Pin_12), PSOrient1.12 (Pin_12), R2.2, XBOrient1.12 (Pin_12)
- net RJSH: now reaches M1.9 (A4)
- net RJSH: now also RS1.H2 (H); no longer RT1.3 (VOUT)
- new net: IC6.3 (SW1), Start1.1
- new net: C5.1, U1.1 (REG)
- new net: IC5.10 (IO0_6), IC6.13 (OUT6)
- new net: IC5.11 (IO0_7), IC6.12 (OUT7)
- new net: IC5.13 (IO1_0), IC6.11 (OUT8)
- new net: IC5.4 (IO0_0), IC6.19 (OUT0)
- new net: IC5.5 (IO0_1), IC6.18 (OUT1)
- new net: IC5.6 (IO0_2), IC6.17 (OUT2)
- new net: IC5.7 (IO0_3), IC6.16 (OUT3)
- new net: IC5.8 (IO0_4), IC6.15 (OUT4)
- new net: IC5.9 (IO0_5), IC6.14 (OUT5)
- new net: LRA/ERM1.1 (Pin_1), LRA/ERM1.3 (Pin_3), U1.9 (OUT-)
- new net: LRA/ERM1.2 (Pin_2), LRA/ERM1.4 (Pin_4), U1.7 (OUT+)
- new net: EYESPI1.17 (Pin_17), Ext5.1 (Pin_1)
- new net: EYESPI1.18 (Pin_18), Ext5.3 (Pin_3)
- new net A: A1.2, IC6.7 (SW5)
- new net B: B1.2, IC6.8 (SW6)
- new net D: +D1.2, IC1.7 (SW5), Mate1.5 (Pin_5), PSOrient1.5 (Pin_5), XBOrient1.5 (Pin_5)
- new net GPIO1: Ext4.12 (Pin_12), IC5.15 (IO1_2)
- new net GPIO2: Ext4.10 (Pin_10), IC5.16 (IO1_3)
- new net GPIO3: Ext4.8 (Pin_8), IC5.17 (IO1_4)
- new net GPIO4: Ext4.6 (Pin_6), IC5.18 (IO1_5)
- new net GPIO5: Ext4.4 (Pin_4), IC5.19 (IO1_6)
- new net GPIO6: Ext4.2 (Pin_2), IC5.20 (IO1_7)
- new net L: +L1.2, IC1.5 (SW3), Mate1.3 (Pin_3), PSOrient1.3 (Pin_3), XBOrient1.3 (Pin_3)
- new net LB: IC1.2 (SW0), LB1.2
- new net LPDL: IC1.3 (SW1), LPDL1.2, Mate1.1 (Pin_1), PSOrient1.1 (Pin_1), XBOrient1.1 (Pin_1)
- new net OriSelect: IC4.20 (IO1_7), Mate1.6 (Pin_6), PSOrient1.6 (Pin_6)
- new net R: +R1.2, IC1.6 (SW4), Mate1.4 (Pin_4), PSOrient1.4 (Pin_4), XBOrient1.4 (Pin_4)
- new net RB: IC6.6 (SW4), RB1.2
- new net RJSS: IC6.4 (SW2), RS1.B1A (SEL+)
- new net RJSV: M1.10 (A5), RS1.V2 (V)
- new net RPDL: IC6.5 (SW3), RPDL1.2
- new net RTouchProbe: IC5.14 (IO1_1), R1.1
- new net U: +U1.2, IC1.4 (SW2), Mate1.2 (Pin_2), PSOrient1.2 (Pin_2), XBOrient1.2 (Pin_2)
- new net X: IC6.9 (SW7), X1.2
- new net Y: IC6.10 (SW8), Y1.2
- no-connect marks 0 -> 13
Other:
- moved on the sheet: +D1, +L1, +R1, +U1, IC4, LS1, LT1, M1, RS1, RT1
