File: fsckpad-hardware/fsckpad-hardware_revision1.0.kicad_pcb (KiCad board)
At the start: 2 copper layers, 158.1 x 78.3 mm, 55 parts, among them IC1 LS20-S, IC3 ICM-42670-P, IC4 PCA9555D, IC5 PCA9555D, IC6 LS20-S, U1 DRV2605LDGS, X1 1-TS009, Y1 1-TS009

Commit message: Revision 1.0 with haptic driver
Parts:
- removed Bite1, Bite2: Fiducial, JSP_Footprints:6.5mm_MouseBite
- removed C4, C5: 1pF, Capacitor_SMD:C_0603_1608Metric_Pad1.08x0.95mm_HandSolder
- removed Centroid1: Fiducial, Symbol:OSHW-Logo2_24.3x20mm_SilkScreen
- removed LRA/ERM1: Conn_02x02_Odd_Even, Connector_PinHeader_1.00mm:PinHeader_2x02_P1.00mm_Vertical
- removed LRAEnable: 0, Jumper:SolderJumper-2_P1.3mm_Open_TrianglePad1.0x1.5mm
- removed U1: DRV2605LDGS, Package_SO:VSSOP-10_3x3mm_P0.5mm
- C2: value 2.2uf -> 2.2 uf
- C3: value 10nf -> 10 nf
- R4, R5: footprint Resistor_SMD:R_0603_1608Metric_Pad0.98x0.95mm_HandSolder -> Resistor_SMD:R_0603_1608Metric
- moved H3 4.10 mm to (89.8, 64.0)
- moved POW1 3.52 mm to (88.5, 53.2), turned to -90 degrees
- renumbered Feather to M1, Mate to Mate1, PSOrient to PSOrient1, Ext1 to Rumble, XBOrient to XBOrient1
Connections:
- IC4 pad 15: /LRASelect -> unconnected-(IC4-IO1_2-Pad15)
Routing:
- net +3.3V: track 478.2 -> 442.5 mm
- net /SCL: track 215.8 -> 200.5 mm, vias 8 -> 6
- net Net-(LRA/ERM1-Pin_1): track 13.5 -> 0.00 mm, vias 1 -> 0
- net Net-(LRA/ERM1-Pin_2): track 11.9 -> 0.00 mm, vias 1 -> 0
- net /LRASelect: track 8.14 -> 0.00 mm, vias 1 -> 0
- net /RPDL: track 29.1 -> 21.1 mm
- net Net-(U1-REG): track 7.77 -> 0.00 mm
- net GND: track 8.94 -> 3.40 mm, vias 46 -> 34
- net /LT: track 82.2 -> 78.7 mm
- net /PS: track 16.2 -> 18.6 mm
- net /LTouchSense: track 126.9 -> 124.8 mm
- net /SDA: track 225.3 -> 224.0 mm
- net /GPIO2: track 17.4 -> 16.7 mm
- net /GPIO3: track 16.5 -> 17.1 mm
Other:
- board text added: "rev 1.0"
- board text removed: "+"
- board text removed: "J Payne 2024"
- board text removed: "rev 1.0H"
